File: grove/hashlet-grove.kicad_pcb (KiCad board)
At the start: 2 copper layers, 20 x 20 mm, 5 parts, among them P1 TWIG_2.0, U1 ATSHA204A

Commit message: Hashlet for Grove rev v1
Parts:
- added G***: CHIPPAD, CHIPPAD, F.Cu at (202.9, 147.5)
- added G***: CHIPPAD, CHIPPAD, F.Cu at (209.1, 147.5)
- added G***: CHIPPAD, CHIPPAD, F.Cu at (215.0, 147.5)
- added HoleA: P***, 1pin, F.Cu at (210.0, 130.0)
- added HoleB: P***, 1pin, F.Cu at (210.0, 150.0)
- G***: moved to B.Cu
- U1: value ATSHA204A -> ATCRYPTO
- moved G*** 22.3 mm to (216.3, 133.2)
- moved G*** 8.67 mm to (215.9, 146.7)
- moved P1 8.34 mm to (210.0, 136.1)
- moved U1 8.34 mm to (210.2, 142.2)
- moved G*** 5.69 mm to (211.4, 141.4)
Routing:
- added copper zone on B.Cu, net GND
- added copper zone on F.Cu, net GND
Other:
- board size 20 x 20 mm -> 20 x 24.2 mm
- board text added: "AES"
- board text added: "ECC"
- board text added: "Module ID"
- board text added: "SHA"
- board text added: "moonpunch.org"

Commit message: board updated before manufacturing
Routing:
- net GND: track 10.2 -> 22.4 mm, vias 0 -> 1
Other:
- net class Default: via_dia 0.889 -> 0.6; via_drill 0.635 -> 0.4
- rule via_min_drill: 0.508 -> 0.3
- rule via_min_size: 0.889 -> 0.6
Changed lines of the file:
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@@
     (thickness 1.6)
     (drawings 31)
-    (tracks 24)
+    (tracks 32)
     (zones 0)
     (modules 10)
@@
     (22 B.Mask user)
     (23 F.Mask user)
-    (24 Dwgs.User user)
-    (25 Cmts.User user)
-    (26 Eco1.User user)
-    (27 Eco2.User user)
     (28 Edge.Cuts user)
   )
@@
     (segment_width 0.2)
     (edge_width 0.1)
-    (via_size 0.889)
-    (via_drill 0.635)
-    (via_min_size 0.889)
-    (via_min_drill 0.508)
+    (via_size 0.6)
+    (via_drill 0.4)
+    (via_min_size 0.6)
+    (via_min_drill 0.3)
     (uvia_size 0.508)
     (uvia_drill 0.127)
@@
       (drillshape 0)
       (scaleselection 1)
-      (outputdirectory Gergber/))
+      (outputdirectory Gerber/))
   )
   (net 0 "")
@@
     (clearance 0.254)
     (trace_width 0.254)
-    (via_dia 0.889)
-    (via_drill 0.635)
+    (via_dia 0.6)
+    (via_drill 0.4)
     (uvia_dia 0.508)
     (uvia_drill 0.127)
@@
   (segment (start 210.2 139.2) (end 210.2 142.6) (width 0.254) (layer F.Cu) (net 2))
   (segment (start 211 138.4) (end 210.2 139.2) (width 0.254) (layer F.Cu) (net 2))
-  (segment (start 209 136.1) (end 209 138.1) (width 0.254) (layer B.Cu) (net 3))
-  (segment (start 211.205 140.295) (end 212.994 140.295) (width 0.254) (layer F.Cu) (net 3))
-  (segment (start 211.2 140.3) (end 211.205 140.295) (width 0.254) (layer F.Cu) (net 3))
-  (via (at 211.2 140.3) (size 0.889) (layers F.Cu B.Cu) (net 3))
-  (segment (start 209 138.1) (end 211.2 140.3) (width 0.254) (layer B.Cu) (net 3))
+  (segment (start 209 136.1) (end 209 138) (width 0.254) (layer B.Cu) (net 3))
+  (segment (start 211.305 140.295) (end 212.994 140.295) (width 0.254) (layer F.Cu) (net 3))
+  (segment (start 211.3 140.3) (end 211.305 140.295) (width 0.254) (layer F.Cu) (net 3))
+  (via (at 211.3 140.3) (size 0.6) (layers F.Cu B.Cu) (net 3))
+  (segment (start 209 138) (end 211.3 140.3) (width 0.254) (layer B.Cu) (net 3))
+  (segment (start 207 136.1) (end 207 135.8) (width 0.254) (layer B.Cu) (net 4))
+  (via (at 212.5 137.9) (size 0.6) (layers F.Cu B.Cu) (net 4))
+  (segment (start 213.4 137.9) (end 212.5 137.9) (width 0.254) (layer B.Cu) (net 4))
+  (segment (start 214.4 136.9) (end 213.4 137.9) (width 0.254) (layer B.Cu) (net 4))
+  (segment (start 214.4 135.4) (end 214.4 136.9) (width 0.254) (layer B.Cu) (net 4))
+  (segment (start 213.7 134.7) (end 214.4 135.4) (width 0.254) (layer B.Cu) (net 4))
+  (segment (start 208.1 134.7) (end 213.7 134.7) (width 0.254) (layer B.Cu) (net 4))
+  (segment (start 207 135.8) (end 208.1 134.7) (width 0.254) (layer B.Cu) (net 4))
   (segment (start 207 136.1) (end 207 137.4) (width 0.254) (layer F.Cu) (net 4))
   (segment (start 206.105 144.105) (end 207.406 144.105) (width 0.254) (layer F.Cu) (net 4))
